File: Hardware/SparkFun_Pico_Add_On_Flipper.kicad_sch (KiCad schematic)
At the start: 16 parts, among them J1 Conn_01x20, J2 Conn_01x20, J3 Conn_01x20, J4 Conn_01x20, J5 Qwiic_RA, SW1 SMD_RA_5x3mm_h3.6mm

Commit message: Design Review Updates
Widen pads of 1x20 headers
Add "Analog" silk label to ADC pins
Rotate pin labels 180 degrees (more readable when viewing from outside)
Fill out title blocks of schematic and board
Widen traces to 0.01"
Set board constraints, 0.005" copper clearance
Shrink product name in silk and update capitalization
Update ordering notes
Add reset button silk to bottom
Exclude irrelevant DRC warnings/errors
Other:
- company: SparkFun -> SparkFun Electronics
- title: SparkFun Product (Qwiic) -> SparkFun Pico Add-On Flipper
Changed lines of the file:
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@@
 	(paper "USLetter")
 	(title_block
-		(title "SparkFun Product (Qwiic)")
+		(title "SparkFun Pico Add-On Flipper")
+		(date "2025-02-13")
 		(rev "v10")
-		(company "SparkFun")
-		(comment 1 "Designed by: You")
+		(company "SparkFun Electronics")
+		(comment 1 "Designed by: Dryw Wade")
 	)
 	(junction

Commit message: Change reset button
Parts:
- SW1: footprint SparkFun-Switch:Push_SMD_RA_5x3mm -> SparkFun-Switch:Push_SMD_RA_4.5x2.5mm; symbol SparkFun-Switch:SPST_Push_SMD_RA_5x3mm_h3.6mm -> SparkFun-Switch:SPST_Push_SMD_RA_4.5x2.5mm_h3.3mm
Changed lines of the file:
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@@
 	)
 	(symbol
-		(lib_id "SparkFun-Switch:SPST_Push_SMD_RA_5x3mm_h3.6mm")
+		(lib_id "SparkFun-Switch:SPST_Push_SMD_RA_4.5x2.5mm_h3.3mm")
 		(at 129.54 149.86 0)
 		(mirror y)
@@
 			)
 		)
-		(property "Footprint" "SparkFun-Switch:Push_SMD_RA_5x3mm"
+		(property "Footprint" "SparkFun-Switch:Push_SMD_RA_4.5x2.5mm"
 			(at 129.54 154.94 0)
 			(effects

Commit message: Change reset button
Parts:
- J5: footprint SparkFun-Connector:JST_SMD_1.0mm-4_RA -> SparkFun-Connector:JST_SMD_1.0mm-4_Black
- SW1: footprint SparkFun-Switch:Push_SMD_RA_4.5x2.5mm -> SparkFun-Switch:Push_SMD_RA_4.5x3.4mm; symbol SparkFun-Switch:SPST_Push_SMD_RA_4.5x2.5mm_h3.3mm -> SparkFun-Switch:SPST_Push_SMD_RA_4.5x3.4mm_h3.3mm; PROD_ID SWCH-12265 -> SWCH-25434
Changed lines of the file:
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@@
 			)
 		)
-		(property "Footprint" "SparkFun-Connector:JST_SMD_1.0mm-4_RA"
+		(property "Footprint" "SparkFun-Connector:JST_SMD_1.0mm-4_Black"
 			(at 68.58 172.72 0)
 			(effects
@@
 			)
 		)
-		(property "Description" ""
+		(property "Description" "Fiducial Marker"
 			(at 262.89 179.07 0)
 			(effects
@@
 	)
 	(symbol
-		(lib_id "SparkFun-Switch:SPST_Push_SMD_RA_4.5x2.5mm_h3.3mm")
+		(lib_id "SparkFun-Switch:SPST_Push_SMD_RA_4.5x3.4mm_h3.3mm")
 		(at 129.54 149.86 0)
 		(mirror y)
@@
 			)
 		)
-		(property "Footprint" "SparkFun-Switch:Push_SMD_RA_4.5x2.5mm"
+		(property "Footprint" "SparkFun-Switch:Push_SMD_RA_4.5x3.4mm"
 			(at 129.54 154.94 0)
 			(effects
@@
 			)
 		)
-		(property "Datasheet" "~"
+		(property "Datasheet" "https://wmsc.lcsc.com/wmsc/upload/file/pdf/v2/lcsc/2405161820_G-Switch-GT-TC108A-H034-L1S_C22396279.pdf"
 			(at 129.54 160.02 0)
 			(effects
@@
 			)
 		)
-		(property "PROD_ID" "SWCH-12265"
+		(property "PROD_ID" "SWCH-25434"
 			(at 129.54 157.48 0)
 			(effects
@@
 			)
 		)
-		(property "Description" ""
+		(property "Description" "Fiducial Marker"
 			(at 259.08 179.07 0)
 			(effects
@@
 			)
 		)
-		(property "Description" ""
+		(property "Description" "Fiducial Marker"
 			(at 259.08 175.26 0)
 			(effects
@@
 			)
 		)
-		(property "Description" ""
+		(property "Description" "Fiducial Marker"
 			(at 262.89 175.26 0)
 			(effects

Commit message: Update 1x20 header
Parts:
- J1, J2, J3, J4: footprint SparkFun-Connector:1x20_SMD_Pin1Left_Passthru -> SparkFun-Connector:1x20_SMD_Pin1RightUp; symbol SparkFun-Connector:Conn_01x20_SMD_Pin1Left_Passthru -> SparkFun-Connector:Conn_01x20_SMD_Pin1RightUp; PROD_ID CONN-xyz -> CONN-25435
Changed lines of the file:
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@@
 	)
 	(symbol
-		(lib_id "SparkFun-Connector:Conn_01x20_SMD_Pin1Left_Passthru")
+		(lib_id "SparkFun-Connector:Conn_01x20_SMD_Pin1RightUp")
 		(at 210.82 60.96 0)
 		(mirror y)
@@
 			)
 		)
-		(property "Footprint" "SparkFun-Connector:1x20_SMD_Pin1Left_Passthru"
+		(property "Footprint" "SparkFun-Connector:1x20_SMD_Pin1RightUp"
 			(at 210.82 91.44 0)
 			(effects
@@
 			)
 		)
-		(property "Datasheet" "~"
+		(property "Datasheet" "https://wmsc.lcsc.com/wmsc/upload/file/pdf/v2/lcsc/2110100430_XKB-Connection-X6511WVS-20H-C60D48R2_C2883777.pdf"
 			(at 210.82 93.98 0)
 			(effects
@@
 			)
 		)
-		(property "PROD_ID" "CONN-xyz"
+		(property "PROD_ID" "CONN-25435"
 			(at 210.82 99.06 0)
 			(effects
@@
 	)
 	(symbol
-		(lib_id "SparkFun-Connector:Conn_01x20_SMD_Pin1Left_Passthru")
+		(lib_id "SparkFun-Connector:Conn_01x20_SMD_Pin1RightUp")
 		(at 83.82 60.96 0)
 		(mirror y)
@@
 			)
 		)
-		(property "Footprint" "SparkFun-Connector:1x20_SMD_Pin1Left_Passthru"
+		(property "Footprint" "SparkFun-Connector:1x20_SMD_Pin1RightUp"
 			(at 83.82 91.44 0)
 			(effects
@@
 			)
 		)
-		(property "Datasheet" "~"
+		(property "Datasheet" "https://wmsc.lcsc.com/wmsc/upload/file/pdf/v2/lcsc/2110100430_XKB-Connection-X6511WVS-20H-C60D48R2_C2883777.pdf"
 			(at 83.82 93.98 0)
 			(effects
@@
 			)
 		)
-		(property "PROD_ID" "CONN-xyz"
+		(property "PROD_ID" "CONN-25435"
 			(at 83.82 99.06 0)
 			(effects
@@
 	)
 	(symbol
-		(lib_id "SparkFun-Connector:Conn_01x20_SMD_Pin1Left_Passthru")
+		(lib_id "SparkFun-Connector:Conn_01x20_SMD_Pin1RightUp")
 		(at 195.58 60.96 0)
 		(unit 1)
@@
 			)
 		)
-		(property "Footprint" "SparkFun-Connector:1x20_SMD_Pin1Left_Passthru"
+		(property "Footprint" "SparkFun-Connector:1x20_SMD_Pin1RightUp"
 			(at 195.58 91.44 0)
 			(effects
@@
 			)
 		)
-		(property "Datasheet" "~"
+		(property "Datasheet" "https://wmsc.lcsc.com/wmsc/upload/file/pdf/v2/lcsc/2110100430_XKB-Connection-X6511WVS-20H-C60D48R2_C2883777.pdf"
 			(at 195.58 93.98 0)
 			(effects
@@
 			)
 		)
-		(property "PROD_ID" "CONN-xyz"
+		(property "PROD_ID" "CONN-25435"
 			(at 195.58 99.06 0)
 			(effects
@@
 	)
 	(symbol
-		(lib_id "SparkFun-Connector:Conn_01x20_SMD_Pin1Left_Passthru")
+		(lib_id "SparkFun-Connector:Conn_01x20_SMD_Pin1RightUp")
 		(at 68.58 60.96 0)
 		(unit 1)
@@
 		(fields_autoplaced yes)
 		(property "Reference" "J1"
-			(at 68.58 31.75 0)
-			(effects
-				(font
-					(size 1.27 1.27)
-				)
+			(at 71.12 60.9599 0)
+			(effects
+				(font
+					(size 1.27 1.27)
+				)
+				(justify left)
 			)
 		)
 		(property "Value" "Conn_01x20"
-			(at 68.58 34.29 0)
-			(effects
-				(font
-					(size 1.27 1.27)
-				)
-			)
-		)
-		(property "Footprint" "SparkFun-Connector:1x20_SMD_Pin1Left_Passthru"
+			(at 71.12 63.4999 0)
+			(effects
+				(font
+					(size 1.27 1.27)
+				)
+				(justify left)
+			)
+		)
+		(property "Footprint" "SparkFun-Connector:1x20_SMD_Pin1RightUp"
 			(at 68.58 91.44 0)
 			(effects
@@
 			)
 		)
-		(property "Datasheet" "~"
+		(property "Datasheet" "https://wmsc.lcsc.com/wmsc/upload/file/pdf/v2/lcsc/2110100430_XKB-Connection-X6511WVS-20H-C60D48R2_C2883777.pdf"
 			(at 68.58 93.98 0)
 			(effects
@@
 			)
 		)
-		(property "PROD_ID" "CONN-xyz"
+		(property "PROD_ID" "CONN-25435"
 			(at 68.58 99.06 0)
 			(effects

Commit message: Fix "Value" of button in schematic
Parts:
- SW1: value SMD_RA_5x3mm_h3.6mm -> SMD_RA_4.5x3.4mm_h3.3mm
Changed lines of the file:
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@@
 			)
 		)
-		(property "Value" "SMD_RA_5x3mm_h3.6mm"
+		(property "Value" "SMD_RA_4.5x3.4mm_h3.3mm"
 			(at 129.54 144.78 0)
 			(effects

Commit message: Design Review Updates
Fix J1 text location in schematic
Organize ordering notes better
Shrink big vias to match small vias
Nudge button down 0.005"
Changed lines of the file:
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@@
 		(fields_autoplaced yes)
 		(property "Reference" "J1"
-			(at 71.12 60.9599 0)
+			(at 68.58 31.75 0)
 			(effects
 				(font
 					(size 1.27 1.27)
 				)
-				(justify left)
 			)
 		)
 		(property "Value" "Conn_01x20"
-			(at 71.12 63.4999 0)
+			(at 68.58 34.29 0)
 			(effects
 				(font
 					(size 1.27 1.27)
 				)
-				(justify left)
 			)
 		)
